File: hw/MicroTrainer.kicad_pcb (KiCad board)
At the start: 2 copper layers, 134.5 x 118 mm, 42 parts, among them J1 Conn_01x20, J2 Conn_01x20, J4 Conn_01x04, J5 Conn_01x08, SW1 KEY_C, SW10 KEY_B, SW11 KEY_ADDR, SW13 KEY_4, SW14 KEY_5, SW15 KEY_6, SW16 KEY_7, SW17 KEY_STOR, SW18 KEY_STEP, SW19 KEY_0, SW2 KEY_D, SW20 KEY_1, SW21 KEY_2, SW22 KEY_3, SW23 KEY_LOAD, SW24 KEY_RUN, SW3 KEY_E, SW4 KEY_F, SW5 KEY_CLR, SW7 KEY_8, SW8 KEY_9, SW9 KEY_A

Commit message: Staging in preparation of review and ordering
Parts:
- removed J2: Conn_01x20, Connector_PinHeader_2.54mm:PinHeader_1x20_P2.54mm_Vertical
- removed REF** (x8): MountingHole_3.2mm_M3_DIN965_Pad, MountingHole:MountingHole_3.2mm_M3_DIN965_Pad
- added C10: 12pF, Capacitor_SMD:C_0603_1608Metric, F.Cu at (89.0, 34.5)
- added C11: 12pF, Capacitor_SMD:C_0603_1608Metric, F.Cu at (85.2, 37.5)
- added C12: 0.1uF, Capacitor_SMD:C_0603_1608Metric, F.Cu at (89.0, 37.5)
- added C5: 0.1uF, Capacitor_SMD:C_0603_1608Metric, F.Cu at (106.8, 34.5)
- added C6: 0.1uF, Capacitor_SMD:C_0603_1608Metric, F.Cu at (104.7, 44.0)
- added C7: 0.1uF, Capacitor_SMD:C_0603_1608Metric, F.Cu at (95.3, 29.0)
- added C8: 2.2uF, Capacitor_SMD:C_0603_1608Metric, F.Cu at (101.0, 46.8)
- added C9: 2.2uF, Capacitor_SMD:C_0603_1608Metric, F.Cu at (101.0, 49.8)
- added D1: LED, LED_SMD:LED_0805_2012Metric, F.Cu at (111.9, 22.5)
- added D2: LED, LED_SMD:LED_0805_2012Metric, F.Cu at (111.9, 26.5)
- added FID1: Fiducial, Fiducial:Fiducial_1mm_Mask2mm, F.Cu at (31.0, 23.0)
- added FID2: Fiducial, Fiducial:Fiducial_1mm_Mask2mm, F.Cu at (18.0, 118.0)
- added FID3: Fiducial, Fiducial:Fiducial_1mm_Mask2mm, F.Cu at (143.0, 120.0)
- added H1: MountingHole, MountingHole:MountingHole_3.2mm_M3, F.Cu at (17.0, 22.0)
- added H2: MountingHole, MountingHole:MountingHole_3.2mm_M3, F.Cu at (144.0, 22.0)
- added H3: MountingHole, MountingHole:MountingHole_3.2mm_M3, F.Cu at (17.0, 132.0)
- added H4: MountingHole, MountingHole:MountingHole_3.2mm_M3, F.Cu at (144.0, 132.0)
- added H5: MountingHole, MountingHole:MountingHole_3.2mm_M3, F.Cu at (24.5, 23.0)
- added H6: MountingHole, MountingHole:MountingHole_3.2mm_M3, F.Cu at (24.5, 51.5)
- added H7: MountingHole, MountingHole:MountingHole_3.2mm_M3, F.Cu at (76.5, 23.0)
- added H8: MountingHole, MountingHole:MountingHole_3.2mm_M3, F.Cu at (76.5, 51.5)
- added J6: USB_C_Receptacle_USB2.0, Connector_USB:USB_C_Receptacle_G-Switch_GT-USB-7010ASV, F.Cu at (128.8, 22.4)
- added JP1: BootJumper, Jumper:SolderJumper-2_P1.3mm_Open_RoundedPad1.0x1.5mm, F.Cu at (107.2, 22.5)
- added R10: 330, Resistor_SMD:R_0603_1608Metric, F.Cu at (115.5, 22.5)
- added R11: 330, Resistor_SMD:R_0603_1608Metric, F.Cu at (115.5, 26.5)
- added R12: 5.1k, Resistor_SMD:R_0603_1608Metric, F.Cu at (97.3, 49.8)
- added R5: 5.1k, Resistor_SMD:R_0603_1608Metric, F.Cu at (131.8, 32.5)
- added R6: 5.1k, Resistor_SMD:R_0603_1608Metric, F.Cu at (128.0, 32.5)
- added R7: 10, Resistor_SMD:R_0603_1608Metric, F.Cu at (128.0, 29.5)
- added R8: 10, Resistor_SMD:R_0603_1608Metric, F.Cu at (131.8, 29.5)
- added R9: 5.1k, Resistor_SMD:R_0603_1608Metric, F.Cu at (107.1, 26.5)
- added SW25: KEY_RST, Button_Switch_Keyboard:SW_Cherry_MX_1.00u_PCB, F.Cu at (133.0, 79.9)
- added U1: LP5907MFX-3.3, Package_TO_SOT_SMD:SOT-23-5, F.Cu at (119.5, 30.9)
- added U3: STM32F411R_C-E_Tx, Package_QFP:LQFP-64_10x10mm_P0.5mm, F.Cu at (97.8, 37.8)
- added Y1: 25MHz, Crystal:Crystal_SMD_3225-4Pin_3.2x2.5mm, F.Cu at (84.6, 33.6)
- C1, C3: value 1uF -> 2.2uF; footprint Capacitor_THT:C_Rect_L7.0mm_W4.5mm_P5.00mm -> Capacitor_SMD:C_0603_1608Metric
- C2, C4: footprint Capacitor_THT:C_Rect_L7.0mm_W4.5mm_P5.00mm -> Capacitor_SMD:C_0603_1608Metric
- J1: value Conn_01x20 -> Conn_ARM_SWD_TagConnect_TC2030; footprint Connector_PinHeader_2.54mm:PinHeader_1x20_P2.54mm_Vertical -> Connector:Tag-Connect_TC2030-IDC-FP_2x03_P1.27mm_Vertical; moved to B.Cu
- J4: footprint Connector_PinHeader_2.54mm:PinHeader_1x04_P2.54mm_Vertical -> Connector_PinSocket_2.54mm:PinSocket_1x04_P2.54mm_Vertical
- J5: footprint Connector_PinHeader_2.54mm:PinHeader_1x08_P2.54mm_Vertical -> Connector_PinSocket_2.54mm:PinSocket_1x08_P2.54mm_Vertical
- R1, R2, R3, R4: value 4.7k -> 5.1k; footprint Resistor_THT:R_Axial_DIN0207_L6.3mm_D2.5mm_P10.16mm_Horizontal -> Resistor_SMD:R_0603_1608Metric
- moved J1 80.3 mm to (54.5, 37.5), turned to 180 degrees
- moved C3 33.4 mm to (119.3, 26.5)
- moved C1 17.4 mm to (123.8, 29.5)
- moved R2 17.2 mm to (125.8, 63.0), turned to 0 degrees
- moved C2 15.1 mm to (123.8, 32.5)
- moved R4 11.3 mm to (125.8, 69.0), turned to 0 degrees
- moved C4 8.49 mm to (89.0, 40.5)
- moved R3 6.57 mm to (125.8, 66.0), turned to 0 degrees
- moved R1 2.67 mm to (125.7, 60.0), turned to 0 degrees
- moved SW24 0.47 mm to (133.0, 120.0)
- moved SW1 0.47 mm to (33.0, 60.0)
- moved SW13 0.47 mm to (33.0, 100.0)
- moved SW19 0.47 mm to (33.0, 120.0)
- moved SW2 0.47 mm to (53.0, 60.0)
- moved SW20 0.47 mm to (53.0, 120.0)
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Connections:
- J1 pad 1: /PB12SDCS -> +3V3
- J1 pad 2: /PB13SCK -> /SWDIO
- J1 pad 3: /PB14MISO -> /NRST
- J1 pad 4: /PB15MOSI -> /SWCLK
- J1 pad 5: /PA8 -> GND
- J1 pad 6: /PA9 -> unconnected-(J1-SWO-Pad6)
- J5 pad 3: /PB9LCDCS -> /PB10LCDCS
- J5 pad 4: /PC15LCDRST -> /PB7LCDRST
- J5 pad 5: /PC14LCDA0 -> /PB6LCDA0
- R1 pad 1: /PB3 -> /PC6
- R2 pad 1: /PB4 -> /PC7
- R3 pad 1: /PB5 -> /PC8
- R4 pad 1: /PB6 -> /PC9
- SW1 pad 1: /PB3 -> /PC6
- SW1 pad 2: /PA8 -> /PA5
- SW10 pad 1: /PB4 -> /PC7
- SW10 pad 2: /PA11 -> /PA2
- SW11 pad 1: /PB4 -> /PC7
- SW11 pad 2: /PA12 -> /PA1
- SW13 pad 1: /PB5 -> /PC8
- SW13 pad 2: /PA8 -> /PA5
- SW14 pad 1: /PB5 -> /PC8
- SW14 pad 2: /PA9 -> /PA4
- SW15 pad 1: /PB5 -> /PC8
- SW15 pad 2: /PA10 -> /PA3
- SW16 pad 1: /PB5 -> /PC8
- SW16 pad 2: /PA11 -> /PA2
- SW17 pad 1: /PB5 -> /PC8
- SW17 pad 2: /PA12 -> /PA1
- SW18 pad 1: /PB5 -> /PC8
- SW18 pad 2: /PA15 -> /PA0
- SW19 pad 1: /PB6 -> /PC9
- SW19 pad 2: /PA8 -> /PA5
- SW2 pad 1: /PB3 -> /PC6
- SW2 pad 2: /PA9 -> /PA4
- SW20 pad 1: /PB6 -> /PC9
- SW20 pad 2: /PA9 -> /PA4
- SW21 pad 1: /PB6 -> /PC9
- SW21 pad 2: /PA10 -> /PA3
- SW22 pad 1: /PB6 -> /PC9
- SW22 pad 2: /PA11 -> /PA2
- SW23 pad 1: /PB6 -> /PC9
- SW23 pad 2: /PA12 -> /PA1
- SW24 pad 1: /PB6 -> /PC9
- SW24 pad 2: /PA15 -> /PA0
- SW3 pad 1: /PB3 -> /PC6
- SW3 pad 2: /PA10 -> /PA3
- SW4 pad 1: /PB3 -> /PC6
- SW4 pad 2: /PA11 -> /PA2
- SW5 pad 1: /PB3 -> /PC6
- SW5 pad 2: /PA12 -> /PA1
- SW7 pad 1: /PB4 -> /PC7
- SW7 pad 2: /PA8 -> /PA5
- SW8 pad 1: /PB4 -> /PC7
- SW8 pad 2: /PA9 -> /PA4
- SW9 pad 1: /PB4 -> /PC7
- SW9 pad 2: /PA10 -> /PA3
Routing:
- net /PC9: track 0.00 -> 267.6 mm
- net /PC8: track 0.00 -> 225.3 mm
- net /PA5: track 0.00 -> 186.2 mm, vias 0 -> 3
- net /PC7: track 0.00 -> 181.4 mm
- net /PA4: track 0.00 -> 164.1 mm, vias 0 -> 1
- net /PC6: track 0.00 -> 150.9 mm
- net /PA3: track 0.00 -> 142.3 mm, vias 0 -> 1
- net /PA1: track 0.00 -> 125.0 mm, vias 0 -> 3
- net /PA2: track 0.00 -> 122.6 mm, vias 0 -> 1
- net /NRST: track 0.00 -> 118.8 mm, vias 0 -> 1
- net /PA0: track 0.00 -> 118.8 mm, vias 0 -> 3
- net /PB15MOSI: track 0.00 -> 94.1 mm, vias 0 -> 3
- net /PB13SCK: track 0.00 -> 91.0 mm, vias 0 -> 3
- net /PB6LCDA0: track 0.00 -> 85.9 mm, vias 0 -> 2
- net /PB7LCDRST: track 0.00 -> 85.1 mm, vias 0 -> 2
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- added copper zone on F.Cu, net +3V3
- added copper zone on In2.Cu, net +3V3
- added copper zone on F.Cu, net +5V
- added copper zone on In2.Cu, net +5V
- added copper zone on B.Cu, net GND
- added copper zone on F.Cu, net GND
- added copper zone on In1.Cu, net GND
Other:
- board size 134.5 x 118 mm -> 135 x 118 mm
- copper layers 2 -> 4
- net class Default removed
- board text added: "+"
- board text added: "ARM Microprocessor Trainer, Copyright 2021-2023, M. Lyle. Revision B"
- board text removed: "ARM Microprocessor Trainer, Copyright 2021, M. Lyle. Revision A"
